Commit message: changed mesh refs in urdf to point to dynamixel_urdf package

File: urdf/ax12.xacro (robot description, xacro)
@@ -20,5 +20,5 @@
         <origin xyz=" 0 0 0 " rpy="1.57 0 1.57" />
         <geometry>
-          <mesh filename="package://maxwell_defs/meshes/ax12.stl" scale="0.001 0.001 0.001"/>
+          <mesh filename="package://dynamixel_urdf/meshes/ax12.stl" scale="0.001 0.001 0.001"/>
         </geometry>
         <material name="${color}"/>
@@ -49,5 +49,5 @@
         <origin xyz=" 0 0 0 " rpy="0 0 0" />
         <geometry>
-          <mesh filename="package://maxwell_defs/meshes/ax12.stl" scale="0.001 0.001 0.001"/>
+          <mesh filename="package://dynamixel_urdf/meshes/ax12.stl" scale="0.001 0.001 0.001"/>
         </geometry>
         <material name="${color}"/>
@@ -80,5 +80,5 @@
         <origin xyz=" 0 0 0 " rpy="3.14 0 0" />
         <geometry>
-          <mesh filename="package://maxwell_defs/meshes/F3.stl" scale="0.001 0.001 0.001"/>
+          <mesh filename="package://dynamixel_urdf/meshes/F3.stl" scale="0.001 0.001 0.001"/>
         </geometry>
         <material name="${color}"/>
@@ -109,5 +109,5 @@
         <origin xyz=" 0 0 0 " rpy="0 0 0" />
         <geometry>
-          <mesh filename="package://maxwell_defs/meshes/F3.stl" scale="0.001 0.001 0.001"/>
+          <mesh filename="package://dynamixel_urdf/meshes/F3.stl" scale="0.001 0.001 0.001"/>
         </geometry>
         <material name="${color}"/>
@@ -140,5 +140,5 @@
         <origin xyz=" 0 0 0 " rpy="0 0 0" />
         <geometry>
-          <mesh filename="package://maxwell_defs/meshes/F2.stl" scale="0.001 0.001 0.001"/>
+          <mesh filename="package://dynamixel_urdf/meshes/F2.stl" scale="0.001 0.001 0.001"/>
         </geometry>
         <material name="${color}"/>
@@ -171,5 +171,5 @@
         <origin xyz=" 0 0 0 " rpy="3.14 0 0" />
         <geometry>
-          <mesh filename="package://maxwell_defs/meshes/F1.stl" scale="1 1 1"/>
+          <mesh filename="package://dynamixel_urdf/meshes/F1.stl" scale="1 1 1"/>
         </geometry>
         <material name="${color}"/>
@@ -200,5 +200,5 @@
         <origin xyz=" 0 0 0 " rpy="3.14 0 0" />
         <geometry>
-          <mesh filename="package://maxwell_defs/meshes/F6.stl" scale="1 1 1"/>
+          <mesh filename="package://dynamixel_urdf/meshes/F6.stl" scale="1 1 1"/>
         </geometry>
         <material name="${color}"/>
@@ -229,5 +229,5 @@
         <origin xyz="0 0 0" rpy="0 0 0" />
         <geometry>
-          <mesh filename="package://maxwell_defs/meshes/F9.stl" scale="1 1 1"/>
+          <mesh filename="package://dynamixel_urdf/meshes/F9.stl" scale="1 1 1"/>
         </geometry>
         <material name="${color}"/>
@@ -258,5 +258,5 @@
         <origin xyz="0 0 0" rpy="0 0 0" />
         <geometry>
-          <mesh filename="package://maxwell_defs/meshes/F11.stl" scale="1 1 1"/>
+          <mesh filename="package://dynamixel_urdf/meshes/F11.stl" scale="1 1 1"/>
         </geometry>
         <material name="${color}"/>

File: urdf/rx28.xacro (robot description, xacro)
@@ -18,5 +18,5 @@
         <origin xyz=" 0 0 0 " rpy="0 0 -1.57" />
         <geometry>
-          <mesh filename="package://maxwell_defs/meshes/rx28.stl" scale="1 1 1"/>
+          <mesh filename="package://dynamixel_urdf/meshes/rx28.stl" scale="1 1 1"/>
         </geometry>
         <material name="${color}"/>
@@ -47,5 +47,5 @@
         <origin xyz=" 0 0 0 " rpy="1.57 1.57 0" />
         <geometry>
-          <mesh filename="package://maxwell_defs/meshes/rx28.stl" scale="1 1 1"/>
+          <mesh filename="package://dynamixel_urdf/meshes/rx28.stl" scale="1 1 1"/>
         </geometry>
         <material name="${color}"/>
@@ -78,5 +78,5 @@
         <origin xyz=" 0 0 0 " rpy="-1.57 -1.57 0" />
         <geometry>
-          <mesh filename="package://maxwell_defs/meshes/rx28-side-bracket.stl" scale="1 1 1"/>
+          <mesh filename="package://dynamixel_urdf/meshes/rx28-side-bracket.stl" scale="1 1 1"/>
         </geometry>
         <material name="${color}"/>
@@ -107,5 +107,5 @@
         <origin xyz=" 0 0 0 " rpy="1.57 1.57 0" />
         <geometry>
-          <mesh filename="package://maxwell_defs/meshes/rx28-side-bracket.stl" scale="1 1 1"/>
+          <mesh filename="package://dynamixel_urdf/meshes/rx28-side-bracket.stl" scale="1 1 1"/>
         </geometry>
         <material name="${color}"/>
@@ -138,5 +138,5 @@
         <origin xyz="0 0 0" rpy="0 0 -1.57" />
         <geometry>
-          <mesh filename="package://maxwell_defs/meshes/rx28-hinge-bracket.stl" scale="1 1 1"/>
+          <mesh filename="package://dynamixel_urdf/meshes/rx28-hinge-bracket.stl" scale="1 1 1"/>
         </geometry>
         <material name="${color}"/>

File: urdf/rx64.xacro (robot description, xacro)
@@ -18,5 +18,5 @@
         <origin xyz=" 0 0 0 " rpy="0 0 -1.57" />
         <geometry>
-          <mesh filename="package://maxwell_defs/meshes/rx64.stl" scale="1 1 1"/>
+          <mesh filename="package://dynamixel_urdf/meshes/rx64.stl" scale="1 1 1"/>
         </geometry>
         <material name="${color}"/>
@@ -47,5 +47,5 @@
         <origin xyz=" 0 0 0 " rpy="1.57 1.57 0" />
         <geometry>
-          <mesh filename="package://maxwell_defs/meshes/rx64.stl" scale="1 1 1"/>
+          <mesh filename="package://dynamixel_urdf/meshes/rx64.stl" scale="1 1 1"/>
         </geometry>
         <material name="${color}"/>
@@ -78,5 +78,5 @@
         <origin xyz=" 0 0 0 " rpy="1.57 0 0" />
         <geometry>
-          <mesh filename="package://maxwell_defs/meshes/rx64-side-bracket.stl" scale="1 1 1"/>
+          <mesh filename="package://dynamixel_urdf/meshes/rx64-side-bracket.stl" scale="1 1 1"/>
         </geometry>
         <material name="${color}"/>
@@ -109,5 +109,5 @@
         <origin xyz="0 0 0" rpy="0 0 -1.57" />
         <geometry>
-          <mesh filename="package://maxwell_defs/meshes/rx64-hinge-bracket.stl" scale="1 1 1"/>
+          <mesh filename="package://dynamixel_urdf/meshes/rx64-hinge-bracket.stl" scale="1 1 1"/>
         </geometry>
         <material name="${color}"/>

Commit message: added axis param to ax12_side_revolute

File: urdf/ax12.xacro (robot description, xacro)
@@ -61,8 +61,8 @@
     </link>
   </macro>
-  <macro name="ax12_side_revolute" params="name parent llimit ulimit vlimit color *origin" >
+  <macro name="ax12_side_revolute" params="name parent llimit ulimit vlimit color axis *origin" >
     <joint name="${name}_joint" type="revolute">
       <insert_block name="origin" />
-      <axis xyz="0 0 1"/>
+      <axis xyz="${axis}"/>
       <limit effort="30" velocity="${vlimit}" lower="${llimit}" upper="${ulimit}" />
       <parent link="${parent}"/>
